File: PCB/XDQ-001.kicad_pcb (KiCad board)
At the start: 4 copper layers, 45 x 50 mm, 66 parts, among them J1 RADIO, J2 ESC, J3 GPS, J4 SWD, J5 USB_B_Micro, J6 BEC CONECTOR, U1 USBLC6-2P6, U2 AP2112K-3.3, U3 STM32F411CEUx, U4 AP2112K-3.3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

Commit message: feat: initialize project directory with KiCad design files, firmware, and reference documentation
Parts:
- J1: footprint Connector_PinSocket_2.54mm:PinSocket_1x10_P2.54mm_Vertical -> huellas_simplificadas:SolderWirePad_1x10_SMD_1.5x3mm
- J2: footprint Connector_PinSocket_2.54mm:PinSocket_1x05_P2.54mm_Vertical -> huellas_simplificadas:SolderWirePad_1x05_SMD_1.5x3mm
- J3, J4: footprint Connector_PinSocket_2.54mm:PinSocket_1x04_P2.54mm_Vertical -> Connector_JST:JST_PH_B4B-PH-K_1x04_P2.00mm_Vertical
- moved J1 11.5 mm to (91.0, 94.8)
- moved J2 5.05 mm to (118.0, 122.0)
- moved J3 2.72 mm to (130.2, 112.5), turned to 90 degrees
- moved J4 1.68 mm to (98.2, 120.5), turned to 0 degrees
- moved C1 1.58 mm to (103.2, 117.8)
Routing:
- net /SWDIO: track 12.5 -> 10.7 mm
- net GND: track 143.8 -> 142.3 mm, vias 29 -> 31
- net /GPS_RX: track 36.3 -> 34.9 mm
- net /GPS_TX: track 38.3 -> 37.2 mm
- net /SWCLK: track 9.43 -> 8.51 mm
- net /NRST: track 22.8 -> 23.4 mm
