File: PCB/XDQ-001.kicad_sch (KiCad schematic)
At the start: 62 parts, among them J1 RADIO, J2 ESC, J3 GPS, J4 SWD, J5 USB_B_Micro, J6 BEC CONECTOR, U1 USBLC6-2P6, U2 AP2112K-3.3, U3 STM32F411CEUx, U4 AP2112K-3.3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

Commit message: feat: initialize project directory with KiCad design files, firmware, and reference documentation
Parts:
- J1: footprint Connector_PinSocket_2.54mm:PinSocket_1x10_P2.54mm_Vertical -> huellas_simplificadas:SolderWirePad_1x10_SMD_1.5x3mm
- J2: footprint Connector_PinSocket_2.54mm:PinSocket_1x05_P2.54mm_Vertical -> huellas_simplificadas:SolderWirePad_1x05_SMD_1.5x3mm
- J3, J4: footprint Connector_PinSocket_2.54mm:PinSocket_1x04_P2.54mm_Vertical -> Connector_JST:JST_PH_B4B-PH-K_1x04_P2.00mm_Vertical
Changed lines of the file:
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@@
 			)
 		)
-		(property "Footprint" "Connector_PinSocket_2.54mm:PinSocket_1x05_P2.54mm_Vertical"
+		(property "Footprint" "huellas_simplificadas:SolderWirePad_1x05_SMD_1.5x3mm"
 			(at 20.32 99.06 0)
 			(effects
@@
 			)
 		)
-		(property "Footprint" "Connector_PinSocket_2.54mm:PinSocket_1x04_P2.54mm_Vertical"
+		(property "Footprint" "Connector_JST:JST_PH_B4B-PH-K_1x04_P2.00mm_Vertical"
 			(at 20.32 177.8 0)
 			(effects
@@
 			)
 		)
-		(property "Footprint" "Connector_PinSocket_2.54mm:PinSocket_1x04_P2.54mm_Vertical"
+		(property "Footprint" "Connector_JST:JST_PH_B4B-PH-K_1x04_P2.00mm_Vertical"
 			(at 20.32 120.65 0)
 			(effects
@@
 			)
 		)
-		(property "Footprint" "Connector_PinSocket_2.54mm:PinSocket_1x10_P2.54mm_Vertical"
+		(property "Footprint" "huellas_simplificadas:SolderWirePad_1x10_SMD_1.5x3mm"
 			(at 20.32 76.2 0)
 			(effects
