File: PCB/XDQ-001.kicad_sch (KiCad schematic)
At the start: 62 parts, among them J1 RADIO, J2 ESC, J3 GPS, J4 SWD, J5 USB_B_Micro, J6 BEC CONECTOR, U1 USBLC6-2P6, U2 AP2112K-3.3, U3 STM32F411CEUx, U4 AP2112K-3.3, U5 W25Q32JVSS, U6 AP2112K-3.3, U7 ICM-42688-P, U8 BMP280, U9 MMC5983MA, Y1 8Mhz

Commit message: Updated FCB and documentation
Parts:
- J5: footprint Connector_USB:USB_Micro-B_Molex-105017-0001 -> huellas_simplificadas:USB_Micro-B_GCT_USB3076-30-A
Changed lines of the file:
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@@
 			)
 		)
-		(property "Footprint" "Connector_USB:USB_Micro-B_Molex-105017-0001"
+		(property "Footprint" "huellas_simplificadas:USB_Micro-B_GCT_USB3076-30-A"
 			(at 25.4 149.86 0)
 			(hide yes)
